File: isa_svga.sch (KiCad schematic (older format))
At the start: 62 parts, among them P1 VGA, U1 TVGA9000i, U2 27C256, U3 256Kx4 70ns, U4 256Kx4 70ns, U5 256Kx4 70ns, U6 256Kx4 70ns, X1 40MHz

Commit message: Add files via upload
Parts:
- removed BUS1: BUSPC_DEV, Custom:Conn_Bus_ISA8_TVGA, symbol isa_svga-rescue:BUSPC_DEV
- removed JP1: HSYNC_SEL, Connector_PinHeader_2.54mm:PinHeader_1x02_P2.54mm_Vertical, symbol isa_svga-rescue:JUMPER
- removed P1: VGA, Custom:DSUB-15-HD_Female_Horizontal_CONNFLY_DS1308, symbol isa_svga-rescue:DE15
- added J1: PC104, Custom:PC104_Platform, symbol Connector_Generic_MountingPin:Conn_02x32_Odd_Even_MountingPin
- added J2: Jumper for 8-bit bus, Custom:Triple-bridged-jumper, symbol Connector_Generic:Conn_02x03_Odd_Even
- added J3: PC104_16, Connector_PinSocket_2.54mm:PinSocket_2x20_P2.54mm_Vertical, symbol Connector_Generic:Conn_02x20_Odd_Even
- added J4: VGA Output, Connector_IDC:IDC-Header_2x05_P2.54mm_Horizontal, symbol Connector_Generic:Conn_02x05_Odd_Even
- added JP4: ALE_Source, Jumper:SolderJumper-3_P1.3mm_Bridged12_Pad1.0x1.5mm, symbol Jumper:SolderJumper_3_Bridged12
- added NT7: NetTie, NetTie:NetTie-2_SMD_Pad0.5mm, symbol Device:Net-Tie_2
- added SW1: VGA Config, Button_Switch_THT:SW_DIP_SPSTx02_Slide_9.78x7.26mm_W7.62mm_P2.54mm, symbol Switch:SW_DIP_x02
- C1, C10, C11, C12, C2, C3, C4, C5, C6, C7, C8, C9: value 100nF -> 104; footprint Capacitor_THT:C_Disc_D4.3mm_W1.9mm_P5.00mm -> Custom KiCad Library:C_0603_1608Metric
- C13, C14, C15, C16: value 10uF -> 106; footprint Capacitor_THT:CP_Radial_Tantal_D4.5mm_P5.00mm -> Custom KiCad Library:C_0603_1608Metric
- C17: value 1nF -> 102; footprint Capacitor_THT:C_Disc_D4.3mm_W1.9mm_P5.00mm -> Custom KiCad Library:C_0805_2012Metric
- C18: value 470pF -> 471; footprint Capacitor_THT:C_Disc_D4.3mm_W1.9mm_P5.00mm -> Custom KiCad Library:C_0805_2012Metric
- C19: value 100pF -> 101; footprint Capacitor_THT:C_Disc_D4.3mm_W1.9mm_P5.00mm -> Custom KiCad Library:C_0805_2012Metric
- C20, C21, C22, C23, C24, C25, C26, C27: value 47pF -> 47; footprint Capacitor_THT:C_Disc_D4.3mm_W1.9mm_P5.00mm -> Custom KiCad Library:C_0603_1608Metric
- FB1, FB2, FB3, FB4, FB5, FB6: footprint Resistor_THT:R_Axial_DIN0204_L3.6mm_D1.6mm_P7.62mm_Horizontal -> Custom KiCad Library:C_0805_2012Metric
- L1, L3: value 5.7uH -> 5.6uH; footprint Resistor_THT:R_Axial_DIN0207_L6.3mm_D2.5mm_P7.62mm_Horizontal -> Custom KiCad Library:C_0805_2012Metric
- L2: footprint Resistor_THT:R_Axial_DIN0207_L6.3mm_D2.5mm_P7.62mm_Horizontal -> Custom KiCad Library:C_0805_2012Metric
- R1, R10, R14, R15, R16, R2, R3, R4, R8, R9: footprint Resistor_THT:R_Axial_DIN0207_L6.3mm_D2.5mm_P7.62mm_Horizontal -> Custom KiCad Library:R_0805_2012Metric
- R11, R12, R13: value 150 -> 4.7K; footprint Resistor_THT:R_Axial_DIN0207_L6.3mm_D2.5mm_P7.62mm_Horizontal -> Custom KiCad Library:R_0805_2012Metric
- R5, R6, R7: value 4.7K -> 150; footprint Resistor_THT:R_Axial_DIN0207_L6.3mm_D2.5mm_P7.62mm_Horizontal -> Custom KiCad Library:R_0805_2012Metric
- U1: footprint Custom:PQFP-160 -> Custom KiCad Library:PQFP-160_28x28mm_P0.65mm_LongPads
- U2: footprint Package_DIP:DIP-28_W15.24mm_Socket -> Custom KiCad Library:DIP-28_W15.24mm_Socket
- U3, U4, U5, U6: footprint Package_DIP:DIP-20_W7.62mm_Socket -> Custom KiCad Library:DIP-20_W7.62mm_Socket
- Y1: renamed from X1; footprint Crystal:Crystal_HC49-4H_Vertical -> Oscillator:Oscillator_SMD_Abracon_ASE-4Pin_3.2x2.5mm; symbol Device:Crystal -> crystal_pin1and3:Crystal_Pin1and3
Connections:
- net A0: now also J1.62 (Pin_62)
- net A1: now also J1.60 (Pin_60)
- net A10: now also J1.42 (Pin_42)
- net A11: now also J1.40 (Pin_40)
- net A12: now also J1.38 (Pin_38)
- net A13: now also J1.36 (Pin_36)
- net A14: now also J1.34 (Pin_34)
- net A15: now also J1.32 (Pin_32)
- net A16: now also J1.30 (Pin_30)
- net A17: now also J1.28 (Pin_28), J2.1 (Pin_1); no longer U1.113 (SA17(LA17))
- net A18: now also J1.26 (Pin_26), J2.3 (Pin_3); no longer U1.114 (SA18(LA18))
- net A19: now also J1.24 (Pin_24), J2.5 (Pin_5); no longer U1.115 (SA19(LA19))
- net A2: now also J1.58 (Pin_58)
- net A3: now also J1.56 (Pin_56)
- net A4: now also J1.54 (Pin_54)
- net A5: now also J1.52 (Pin_52)
- net A6: now also J1.50 (Pin_50)
- net A7: now also J1.48 (Pin_48)
- net A8: now also J1.46 (Pin_46)
- net A9: now also J1.44 (Pin_44)
- net AEN: now also J1.22 (Pin_22)
- net B: now also R5.1; no longer R13.1
- net D0: now also J1.18 (Pin_18)
- net D1: now also J1.16 (Pin_16)
- net D2: now also J1.14 (Pin_14)
- net D3: now also J1.12 (Pin_12)
- net D4: now also J1.10 (Pin_10)
- net D5: now also J1.8 (Pin_8)
- net D6: now also J1.6 (Pin_6)
- net D7: now also J1.4 (Pin_4)
- net G: now also R6.1; no longer R12.1
- net GND: now also C17.1, C26.1, C27.1, J1.1 (Pin_1), J1.61 (Pin_61), J1.63 (Pin_63), J1.64 (Pin_64), J1.MP (MountPin), J3.1 (Pin_1), J3.2 (Pin_2), J3.38 (Pin_38), J3.40 (Pin_40), J4.8 (Pin_8), NT7.1; no longer C17.2, C23.2, C24.2, C25.2, C26.2, C27.2, R10.2, R5.2, R7.2, U1.1 (AVSS2)
- net HSYNC: now also FB4.1; no longer FB4.2
- net IOCHRDY: now also J1.20 (Pin_20)
- net MD2: now also SW1.2; no longer R6.1
- net MD3: now also R4.1; no longer R7.1
- net MD7: now also R12.1; no longer R2.1
- net MONITOR: now also FB6.1; no longer FB6.2
- net OSC: now also J1.59 (Pin_59)
- net R: now also R7.1; no longer R11.1
- net RESET: now also J1.3 (Pin_3)
- net RMD1: now also SW1.1; no longer R5.1
- net RMD4: now also R13.1; no longer R4.1
- net RMD6: now also R11.1; no longer R3.1
- net VCC: now also J1.5 (Pin_5), J1.57 (Pin_57), J3.34 (Pin_34), JP4.3 (B); no longer U1.21 (ALE)
- net VSYNC: now also FB5.1; no longer FB5.2
- net ~IOR: now also J1.27 (Pin_27)
- net ~IOW: now also J1.25 (Pin_25)
- net ~MEMR: now also J1.23 (Pin_23)
- net ~MEMW: now also J1.21 (Pin_21)
- net ~NMI: now also J1.2 (Pin_2)
- net ~REFRESH: now also J1.37 (Pin_37)
- net ~MEMCS16: now reaches R1.1, U1.102 (~MCS16)
- net ~MEMCS16: now also J3.4 (Pin_4)
- net D15: now reaches U1.103 (SD15)
- net D15: now also J3.37 (Pin_37)
- net D14: now reaches U1.104 (SD14)
- net D14: now also J3.35 (Pin_35)
- net D13: now reaches U1.105 (SD13)
- net D13: now also J3.33 (Pin_33)
- net D12: now reaches U1.106 (SD12)
- net D12: now also J3.31 (Pin_31)
- net D11: now reaches U1.107 (SD11)
- net D11: now also J3.29 (Pin_29)
- net D10: now reaches U1.108 (SD10)
- net D10: now also J3.27 (Pin_27)
- net D9: now reaches U1.109 (SD9)
- net D9: now also J3.25 (Pin_25)
- net D8: now reaches U1.110 (SD8)
- net D8: now also J3.23 (Pin_23)
- net LA20: now reaches U1.116 (LA20)
- net LA20: now also J3.11 (Pin_11)
- net LA21: now reaches U1.117 (LA21)
- net LA21: now also J3.9 (Pin_9)
- net LA22: now reaches U1.118 (LA22)
- net LA22: now also J3.7 (Pin_7)
- net LA23: now reaches U1.119 (LA23)
- net LA23: now also J3.5 (Pin_5)
- net at L2.2, U1.131 (XTL1): now also Y1.3; no longer Y1.2
- net ~SBHE: now reaches U1.99 (SBHE)
- net ~SBHE: now also J3.3 (Pin_3)
- net DAC_GND: now reaches R6.2
- net DAC_GND: now also C23.1, C24.1, C25.1, R10.2, R5.2, R7.2, U1.1 (AVSS2), J4.2 (Pin_2), J4.4 (Pin_4), J4.6 (Pin_6), NT7.2
- net AVDD1 renamed SYNC_VDD
- net AVDD2 renamed DAC_VDD
- net BLUE renamed xBLUE
- net xBLUE: now also C25.2, J4.1 (Pin_1); no longer C25.1
- net GREEN renamed xGREEN
- net xGREEN: now also C24.2, J4.3 (Pin_3); no longer C24.1
- net RED renamed xRED
- net xRED: now also C23.2, J4.5 (Pin_5); no longer C23.1
- new net: JP4.2 (C), U1.21 (ALE)
- new net: R2.1, SW1.4
- new net: R3.1, SW1.3
- new net ALE: J1.55 (Pin_55), JP4.1 (A)
- new net LA17: J2.2 (Pin_2), J3.17 (Pin_17), U1.113 (SA17(LA17))
- new net LA18: J2.4 (Pin_4), J3.15 (Pin_15), U1.114 (SA18(LA18))
- new net LA19: J2.6 (Pin_6), J3.13 (Pin_13), U1.115 (SA19(LA19))
- new net xHSYNC: C26.2, FB4.2, J4.7 (Pin_7)
- new net xMONITOR: C17.2, FB6.2, J4.10 (Pin_10)
- new net xVSYNC: C27.2, FB5.2, J4.9 (Pin_9)
- no-connect marks 50 -> 52
Other:
- note added: "B A"
- note added: "D C"
- note added: "Switch 1 - Enable VGA\nSwitch 2 - Monitor H-Sync <48.7kHz"
- note removed: "ISA BUS"
- moved on the sheet: C11, C17, C23, C24, C25, C26, C27, FB1, FB2, FB3, FB4, FB5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
